File: kicad/dlp-litho.kicad_sch (KiCad schematic)
At the start: 0 parts

Commit message: Imported sym and footprints of DLP components in TIDA-080010
Other:
- added sheet dmd (dmd.kicad_sch)
Changed lines of the file:
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@@
 	(generator_version "10.0")
 	(paper "A4")
+	(sheet
+		(at 21.59 17.78)
+		(size 17.78 5.08)
+		(exclude_from_sim no)
+		(in_bom yes)
+		(on_board yes)
+		(dnp no)
+		(fields_autoplaced yes)
+		(stroke
+			(width 0.1524)
+			(type solid)
+		)
+		(fill
+			(color 0 0 0 0)
+		)
+		(property "Sheetname" "dmd"
+			(at 21.59 17.0684 0)
+			(show_name no)
+			(do_not_autoplace no)
+			(effects
+				(font
+					(size 1.27 1.27)
+				)
+				(justify left bottom)
+			)
+		)
+		(property "Sheetfile" "dmd.kicad_sch"
+			(at 21.59 23.4446 0)
+			(show_name no)
+			(do_not_autoplace no)
+			(effects
+				(font
+					(size 1.27 1.27)
+				)
+				(justify left top)
+			)
+		)
+		(instances
+			(project "dlp-litho"
+				(path "/d7645be1-b662-48c0-9f1b-489c3df905c3"
+					(page "2")
+				)
+			)
+		)
+	)
 	(sheet_instances
 		(path "/"
